Commit message: Robot Camera and Lidar

File: catkin_ws/src/my_robot/urdf/my_robot.xacro (robot description, xacro)
@@ -7,5 +7,5 @@
     <child link="chassis" />
   </joint>
-  <link name='chassis'>
+  <link name="chassis">
     <pose>0 0 0.1 0 0 0</pose>
     <inertial>
@@ -85,4 +85,5 @@
     <dynamics damping="1.0" friction="1.0"/>
   </joint>
+<!-- Left Wheel -->
   <link name='left_wheel'>
     <inertial>
@@ -107,4 +108,5 @@
     </visual>
   </link>
+<!-- Left Wheel Joint -->
   <joint type="continuous" name="left_wheel_hinge">
     <origin xyz="0 0.15 0" rpy="0 0 0"/>
@@ -115,3 +117,66 @@
     <dynamics damping="1.0" friction="1.0"/>
   </joint>
+<!-- Camera -->
+  <link name='camera'>
+    <visual name='camera_visual'>
+      <origin xyz="0 0 0" rpy="0 0 0"/>
+      <geometry>
+        <box size="0.05 0.05 0.05"/>
+      </geometry>
+    </visual>
+    <collision name='camera_colision'>
+      <origin xyz="0 0 0" rpy="0 0 0"/>
+      <geometry>
+        <box size="0.05 0.05 0.05"/>
+      </geometry>
+    </collision>
+    <inertial>
+      <mass value="0.1"/>
+      <box_inertia
+        m="0.1" x="0.05" y="0.05" z="0.05"
+      />
+      <inertia
+       ixx="1e-6" ixy="0" ixz="0"
+       iyy="1e-6" iyz="0"
+       izz="1e-6"
+      />
+    </inertial>
+  </link>
+<!-- Camera Joint -->
+  <joint type="fixed" name="camera_joint">
+    <origin xyz="0.2 0 0" rpy="0 0 0"/>
+    <child link="camera"/>
+    <parent link="chassis"/>
+    <axis xyz="0 1 0" rpy="0 0 0"/>
+  </joint>
+<!-- Lidar Sensor -->
+  <link name="hokuyo">
+    <visual name="hokuyo_visual">
+      <origin xyz="0 0 0" rpy="0 0 0"/>
+      <geometry>
+        <mesh filename="package://my_robot/meshes/hokuyo.dae"/>
+      </geometry>
+    </visual>
+    <collision name="hokuyo_collision">
+      <origin xyz="0 0 0" rpy="0 0 0"/>
+      <geometry>
+        <box size="0.1 0.1 0.1"/>
+      </geometry>
+    </collision>
+    <inertial>
+      <mass value="1e-5"/>
+      <inertia
+       ixx="1e-6" ixy="0" ixz="0"
+       iyy="1e-6" iyz="0"
+       izz="1e-6"
+      />
+    </inertial>
+  </link>
+<!-- Lidar Sensor Joint -->
+  <joint name="hokuyo_joint" type="fixed">
+    <origin xyz="0.15 0 0.1" rpy="0 0 0"/>
+    <parent link="chassis"/>
+    <child link="hokuyo" />
+    <axis xyz="0 1 0" rpy="0 0 0" />
+  </joint>
 </robot>

Commit message: New Robot

File: catkin_ws/src/my_robot/urdf/my_robot.xacro (robot description, xacro)
@@ -22,5 +22,5 @@
       <origin xyz="0 0 0" rpy=" 0 0 0"/>
       <geometry>
-        <box size=".4 .2 .1"/>
+        <box size=".4 .24 .17"/>
       </geometry>
     </collision>
@@ -28,5 +28,5 @@
       <origin xyz="0 0 0" rpy=" 0 0 0"/>
       <geometry>
-        <box size=".4 .2 .1"/>
+        <box size=".4 .24 .17"/>
       </geometry>
     </visual>
@@ -76,4 +76,5 @@
         <cylinder radius="0.1" length="0.05"/>
       </geometry>
+      <material name="red"/>
     </visual>
   </link>
@@ -107,4 +108,5 @@
         <cylinder radius="0.1" length="0.05"/>
       </geometry>
+      <material name="red"/>
     </visual>
   </link>
@@ -118,4 +120,34 @@
     <dynamics damping="1.0" friction="1.0"/>
   </joint>
+<!-- Head -->
+  <link name="head">
+    <visual name="head_visual">
+      <origin xyz="0 0 0" rpy="0 0 1.5707"/>
+      <geometry>
+        <mesh filename="package://my_robot/meshes/head.dae"/>
+      </geometry>
+    </visual>
+    <collision name="head_collision">
+      <origin xyz="0 0 0" rpy="0 0 0"/>
+      <geometry>
+        <box size="0.2 0.2 0.15"/>
+      </geometry>
+    </collision>
+    <inertial>
+      <mass value="1e-5"/>
+      <inertia
+       ixx="0.1" ixy="0" ixz="0"
+       iyy="0.1" iyz="0"
+       izz="0.1"
+      />
+    </inertial>
+  </link>
+<!-- Head Joint -->
+  <joint name="head_joint" type="fixed">
+    <origin xyz="0 0 0.07" rpy="0 0 0"/>
+    <parent link="chassis"/>
+    <child link="head" />
+    <axis xyz="0 1 0" rpy="0 0 0" />
+  </joint>
 <!-- Camera -->
   <link name='camera'>
@@ -146,7 +178,7 @@
 <!-- Camera Joint -->
   <joint type="fixed" name="camera_joint">
-    <origin xyz="0.2 0 0" rpy="0 0 0"/>
+    <origin xyz="0.07 0 0.05" rpy="0 0 0"/>
     <child link="camera"/>
-    <parent link="chassis"/>
+    <parent link="head"/>
     <axis xyz="0 1 0" rpy="0 0 0"/>
   </joint>
@@ -176,6 +208,6 @@
 <!-- Lidar Sensor Joint -->
   <joint name="hokuyo_joint" type="fixed">
-    <origin xyz="0.15 0 0.1" rpy="0 0 0"/>
-    <parent link="chassis"/>
+    <origin xyz="0 0 0.17" rpy="0 0 0"/>
+    <parent link="head"/>
     <child link="hokuyo" />
     <axis xyz="0 1 0" rpy="0 0 0" />
